File: PCB files/motor controller.kicad_pcb (KiCad board)
At the start: 2 copper layers, 84.5 x 62 mm, 29 parts, among them J1 ISP, J2 I2C, J3 Motor Signal, J4 M1, J5 M2, SW1 reset, U1 ATmega328-P, Y1 16Mhz

Commit message: fabrication files ready
Parts:
- moved R6 3.04 mm to (112.5, 75.5)
- moved R7 3.03 mm to (112.5, 73.0)
- moved R8 3.00 mm to (112.5, 70.5)
- moved J1 1.03 mm to (111.2, 91.0)
Routing:
- net GND: track 324.5 -> 321.3 mm
- net /S2: track 3.21 -> 6.25 mm
- net /S3: track 3.20 -> 6.23 mm
- net /S4: track 3.17 -> 6.17 mm
- net /PM2: track 83.4 -> 81.9 mm
- net /RST: track 47.3 -> 45.9 mm
- net Net-(D1-Pad1): track 5.54 -> 6.71 mm
- net +5V: track 150.8 -> 149.8 mm
- net /DM2: track 67.1 -> 66.6 mm

Commit message: generated gerber files
Parts:
- added J6: RST_Jump, Connector_PinHeader_2.54mm:PinHeader_1x01_P2.54mm_Vertical, F.Cu at (110.0, 63.5)
- added J7: RST_Jump, Connector_PinHeader_2.54mm:PinHeader_1x01_P2.54mm_Vertical, F.Cu at (110.0, 86.0)
- added R12: Jumper, Resistor_THT:R_Axial_DIN0207_L6.3mm_D2.5mm_P7.62mm_Horizontal, F.Cu at (76.2, 65.0)
- added R13: Jumper, Resistor_THT:R_Axial_DIN0207_L6.3mm_D2.5mm_P10.16mm_Horizontal, F.Cu at (120.1, 69.1)
- R10, R11: value 10K -> 4.7K
- R5: footprint Resistor_THT:R_Axial_DIN0204_L3.6mm_D1.6mm_P2.54mm_Vertical -> Resistor_THT:R_Axial_DIN0204_L3.6mm_D1.6mm_P5.08mm_Horizontal
- moved C2 5.10 mm to (81.2, 85.5)
- moved C3 5.10 mm to (81.2, 90.5)
- moved Y1 5.10 mm to (87.5, 90.5)
- moved D1 4.00 mm to (76.0, 76.2)
- moved R5 3.39 mm to (89.5, 102.5), turned to 0 degrees
- moved BZ1 2.50 mm to (72.5, 108.2)
- moved J1 2.50 mm to (113.7, 91.0)
- moved R2 2.50 mm to (82.5, 108.8)
- moved R10 1.00 mm to (127.5, 70.3)
- moved R11 1.00 mm to (122.5, 70.5)
Connections:
- J1 pad 5: /RST -> /RST2
- R1 pad 2: /RST -> /RST1
- SW1 pad 1: /RST -> /RST1
- U1 pad 1: /RST -> /RST1
Routing:
- net /RST: track 45.9 -> 0.00 mm
- net /RST1: track 0.00 -> 27.1 mm
- net /PM2: track 81.9 -> 89.0 mm
- net GND: track 321.3 -> 315.4 mm
- net /DM2: track 66.6 -> 72.4 mm
- net Net-(C3-Pad1): track 12.9 -> 18.3 mm
- net /S1: track 9.16 -> 14.6 mm
- net +5V: track 149.8 -> 145.1 mm
- net Net-(C2-Pad1): track 13.0 -> 17.6 mm
- net /RST2: track 0.00 -> 3.74 mm
- net /BUZZ: track 18.4 -> 21.7 mm
- net Net-(D1-Pad1): track 6.71 -> 3.80 mm
- net /SCK: track 4.93 -> 7.43 mm
- net /MISO: track 4.93 -> 7.43 mm
- net /MOSI: track 17.2 -> 19.3 mm
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