File: PCB files/motor controller.kicad_sch (KiCad schematic)
At the start: 29 parts, among them J1 ISP, J2 I2C, J3 Motor Signal, J4 M1, J5 M2, SW1 reset, U1 ATmega328-P, Y1 16Mhz

Commit message: generated gerber files
Parts:
- added J6, J7: RST_Jump, Connector_PinHeader_2.54mm:PinHeader_1x01_P2.54mm_Vertical, symbol Connector:Conn_01x01_Male
- added R12: Jumper, Resistor_THT:R_Axial_DIN0207_L6.3mm_D2.5mm_P7.62mm_Horizontal, symbol Device:R_Small
- added R13: Jumper, Resistor_THT:R_Axial_DIN0207_L6.3mm_D2.5mm_P10.16mm_Horizontal, symbol Device:R_Small
- R10, R11: value 10K -> 4.7K
- R5: footprint Resistor_THT:R_Axial_DIN0204_L3.6mm_D1.6mm_P2.54mm_Vertical -> Resistor_THT:R_Axial_DIN0204_L3.6mm_D1.6mm_P5.08mm_Horizontal
Connections:
- net +5V: now also R12.1, R12.2, R13.1, R13.2
- net RST renamed RST1
- net RST1: now also J6.1 (Pin_1); no longer J1.5 (Pin_5)
- new net RST2: J1.5 (Pin_5), J7.1 (Pin_1)

Commit message: added more jumpers
Parts:
- added J10, J11, J9: 5V, Connector_PinHeader_2.54mm:PinHeader_1x01_P2.54mm_Vertical, symbol Connector:Conn_01x01_Male
- added J8: GND, Connector_PinHeader_2.54mm:PinHeader_1x01_P2.54mm_Vertical, symbol Connector:Conn_01x01_Male
Connections:
- net +5V: now also J10.1 (Pin_1), J11.1 (Pin_1), J9.1 (Pin_1)
- net GND: now also J8.1 (Pin_1)
Changed lines of the file:
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@@
   (junction (at 209.55 72.39) (diameter 0) (color 0 0 0 0)
   )
+  (junction (at 203.2 95.25) (diameter 0) (color 0 0 0 0)
+  )
+  (junction (at 210.82 95.25) (diameter 0) (color 0 0 0 0)
+  )
   (wire (pts (xy 104.14 69.85) (xy 110.49 69.85))
     (stroke (width 0) (type default) (color 0 0 0 0))
   )
+  (wire (pts (xy 209.55 110.49) (xy 212.09 110.49))
+    (stroke (width 0) (type default) (color 0 0 0 0))
+  )
   (wire (pts (xy 45.72 69.85) (xy 53.34 69.85))
     (stroke (width 0) (type default) (color 0 0 0 0))
@@
     (stroke (width 0) (type default) (color 0 0 0 0))
   )
+  (wire (pts (xy 209.55 113.03) (xy 209.55 110.49))
+    (stroke (width 0) (type default) (color 0 0 0 0))
+  )
   (wire (pts (xy 29.21 144.78) (xy 39.37 144.78))
     (stroke (width 0) (type default) (color 0 0 0 0))
@@
     (stroke (width 0) (type default) (color 0 0 0 0))
   )
+  (wire (pts (xy 210.82 88.9) (xy 210.82 95.25))
+    (stroke (width 0) (type default) (color 0 0 0 0))
+  )
   (wire (pts (xy 228.6 72.39) (xy 228.6 68.58))
     (stroke (width 0) (type default) (color 0 0 0 0))
@@
     (stroke (width 0) (type default) (color 0 0 0 0))
   )
+  (wire (pts (xy 203.2 95.25) (xy 210.82 95.25))
+    (stroke (width 0) (type default) (color 0 0 0 0))
+  )
   (wire (pts (xy 104.14 72.39) (xy 110.49 72.39))
     (stroke (width 0) (type default) (color 0 0 0 0))
@@
   )
   (wire (pts (xy 203.2 115.57) (xy 203.2 118.11))
+    (stroke (width 0) (type default) (color 0 0 0 0))
+  )
+  (wire (pts (xy 210.82 95.25) (xy 210.82 101.6))
     (stroke (width 0) (type default) (color 0 0 0 0))
   )
@@
     (pin "1")
   )
+  (symbol (lib_id "Connector:Conn_01x01_Male") (at 215.9 88.9 180) (unit 1)
+    (in_bom yes) (on_board yes)
+    (property "Reference" "J11" (id 0) (at 214.63 83.82 0))
+    (property "Value" "5V" (id 1) (at 215.265 86.36 0))
+    (property "Footprint" "Connector_PinHeader_2.54mm:PinHeader_1x01_P2.54mm_Vertical" (id 2) (at 215.9 88.9 0)
+      (effects (font (size 1.27 1.27)) hide)
+    )
+    (property "Datasheet" "~" (id 3) (at 215.9 88.9 0)
+      (effects (font (size 1.27 1.27)) hide)
+    )
+    (pin "1")
+  )
   (symbol (lib_id "Mechanical:MountingHole_Pad") (at 215.9 66.04 0) (unit 1)
     (in_bom yes) (on_board yes) (fields_autoplaced)
@@
     (pin "2")
   )
+  (symbol (lib_id "Connector:Conn_01x01_Male") (at 215.9 101.6 180) (unit 1)
+    (in_bom yes) (on_board yes) (fields_autoplaced)
+    (property "Reference" "J10" (id 0) (at 215.265 96.52 0))
+    (property "Value" "5V" (id 1) (at 215.265 99.06 0))
+    (property "Footprint" "Connector_PinHeader_2.54mm:PinHeader_1x01_P2.54mm_Vertical" (id 2) (at 215.9 101.6 0)
+      (effects (font (size 1.27 1.27)) hide)
+    )
+    (property "Datasheet" "~" (id 3) (at 215.9 101.6 0)
+      (effects (font (size 1.27 1.27)) hide)
+    )
+    (pin "1")
+  )
   (symbol (lib_id "power:GND") (at 209.55 76.2 0) (unit 1)
     (in_bom yes) (on_board yes) (fields_autoplaced)
@@
     (pin "1")
     (pin "2")
+  )
+  (symbol (lib_name "GND_2") (lib_id "power:GND") (at 209.55 113.03 0) (unit 1)
+    (in_bom yes) (on_board yes) (fields_autoplaced)
+    (property "Reference" "#PWR021" (id 0) (at 209.55 119.38 0)
+      (effects (font (size 1.27 1.27)) hide)
+    )
+    (property "Value" "GND" (id 1) (at 209.55 118.11 0))
+    (property "Footprint" "" (id 2) (at 209.55 113.03 0)
+      (effects (font (size 1.27 1.27)) hide)
+    )
+    (property "Datasheet" "" (id 3) (at 209.55 113.03 0)
+      (effects (font (size 1.27 1.27)) hide)
+    )
+    (pin "1")
   )
   (symbol (lib_id "Connector_Generic:Conn_02x03_Odd_Even") (at 36.83 110.49 0) (unit 1)
@@
     (pin "1")
     (pin "2")
+  )
+  (symbol (lib_id "Connector:Conn_01x01_Male") (at 215.9 95.25 180) (unit 1)
+    (in_bom yes) (on_board yes)
+    (property "Reference" "J9" (id 0) (at 214.63 90.17 0))
+    (property "Value" "5V" (id 1) (at 215.265 92.71 0))
+    (property "Footprint" "Connector_PinHeader_2.54mm:PinHeader_1x01_P2.54mm_Vertical" (id 2) (at 215.9 95.25 0)
+      (effects (font (size 1.27 1.27)) hide)
+    )
+    (property "Datasheet" "~" (id 3) (at 215.9 95.25 0)
+      (effects (font (size 1.27 1.27)) hide)
+    )
+    (pin "1")
   )
   (symbol (lib_id "MCU_Microchip_ATmega:ATmega328-P") (at 88.9 97.79 0) (unit 1)
@@
     (pin "2")
   )
+  (symbol (lib_id "Connector:Conn_01x01_Male") (at 217.17 110.49 180) (unit 1)
+    (in_bom yes) (on_board yes) (fields_autoplaced)
+    (property "Reference" "J8" (id 0) (at 216.535 105.41 0))
+    (property "Value" "GND" (id 1) (at 216.535 107.95 0))
+    (property "Footprint" "Connector_PinHeader_2.54mm:PinHeader_1x01_P2.54mm_Vertical" (id 2) (at 217.17 110.49 0)
+      (effects (font (size 1.27 1.27)) hide)
+    )
+    (property "Datasheet" "~" (id 3) (at 217.17 110.49 0)
+      (effects (font (size 1.27 1.27)) hide)
+    )
+    (pin "1")
+  )
   (symbol (lib_name "+5V_4") (lib_id "power:+5V") (at 203.2 115.57 0) (unit 1)
     (in_bom yes) (on_board yes) (fields_autoplaced)
@@
       (reference "#PWR020") (unit 1) (value "+5V") (footprint "")
     )
+    (path "/76b65430-0dab-40e4-8ba0-5433733f5a05"
+      (reference "#PWR021") (unit 1) (value "GND") (footprint "")
+    )
     (path "/addd7c96-198a-40ec-b8d7-6eb398876d6f"
       (reference "BZ1") (unit 1) (value "Passive") (footprint "Buzzer_Beeper:MagneticBuzzer_ProSignal_ABT-410-RC")
@@
       (reference "J7") (unit 1) (value "RST_Jump") (footprint "Connector_PinHeader_2.54mm:PinHeader_1x01_P2.54mm_Vertical")
     )
+    (path "/df66ce95-2399-404d-8d6a-39b8330d77f2"
+      (reference "J8") (unit 1) (value "GND") (footprint "Connector_PinHeader_2.54mm:PinHeader_1x01_P2.54mm_Vertical")
+    )
+    (path "/8c9998e6-1266-4494-8269-f578c8eb1001"
+      (reference "J9") (unit 1) (value "5V") (footprint "Connector_PinHeader_2.54mm:PinHeader_1x01_P2.54mm_Vertical")
+    )
+    (path "/6445c948-f55c-4d20-b784-33e50711b385"
+      (reference "J10") (unit 1) (value "5V") (footprint "Connector_PinHeader_2.54mm:PinHeader_1x01_P2.54mm_Vertical")
+    )
+    (path "/174ec83d-6715-4022-8c57-ba48b11ee5e1"
+      (reference "J11") (unit 1) (value "5V") (footprint "Connector_PinHeader_2.54mm:PinHeader_1x01_P2.54mm_Vertical")
+    )
     (path "/33aab006-9e39-4482-9a36-fc7df50993d3"

Commit message: backups
Parts:
- removed J10, J11, J9: 5V, Connector_PinHeader_2.54mm:PinHeader_1x01_P2.54mm_Vertical, symbol Connector:Conn_01x01_Male
- removed J6, J7: RST_Jump, Connector_PinHeader_2.54mm:PinHeader_1x01_P2.54mm_Vertical, symbol Connector:Conn_01x01_Male
- removed J8: GND, Connector_PinHeader_2.54mm:PinHeader_1x01_P2.54mm_Vertical, symbol Connector:Conn_01x01_Male
- removed R12: Jumper, Resistor_THT:R_Axial_DIN0207_L6.3mm_D2.5mm_P7.62mm_Horizontal, symbol Device:R_Small
- removed R13: Jumper, Resistor_THT:R_Axial_DIN0207_L6.3mm_D2.5mm_P10.16mm_Horizontal, symbol Device:R_Small
- removed R6, R7, R8, R9: 5K, Resistor_THT:R_Axial_DIN0204_L3.6mm_D1.6mm_P2.54mm_Vertical, symbol Device:R_Small
- added J2: SW, Button_Switch_THT:SW_DIP_SPSTx05_Slide_9.78x14.88mm_W7.62mm_P2.54mm, symbol Connector_Generic:Conn_02x05_Counter_Clockwise
- added R1, R2, R3, R4: 5K, Resistor_SMD:R_0805_2012Metric, symbol Device:R_Small
- C1: footprint Capacitor_THT:CP_Radial_D4.0mm_P2.00mm -> Capacitor_SMD:CP_Elec_6.3x4.5
- C2, C3: footprint Capacitor_THT:C_Disc_D3.4mm_W2.1mm_P2.50mm -> Capacitor_SMD:C_0805_2012Metric
- D1, D2: footprint LED_THT:LED_D3.0mm -> LED_SMD:LED_0805_2012Metric
- R10, R11: footprint Resistor_THT:R_Axial_DIN0207_L6.3mm_D2.5mm_P7.62mm_Horizontal -> Resistor_SMD:R_0805_2012Metric
- R5: footprint Resistor_THT:R_Axial_DIN0204_L3.6mm_D1.6mm_P5.08mm_Horizontal -> Resistor_SMD:R_0805_2012Metric
- R6: renamed from R1; footprint Resistor_THT:R_Axial_DIN0207_L6.3mm_D2.5mm_P7.62mm_Horizontal -> Resistor_SMD:R_0805_2012Metric
- R7: renamed from R2; footprint Resistor_THT:R_Axial_DIN0207_L6.3mm_D2.5mm_P7.62mm_Horizontal -> Resistor_SMD:R_0805_2012Metric
- R8: renamed from R3; footprint Resistor_THT:R_Axial_DIN0207_L6.3mm_D2.5mm_P7.62mm_Horizontal -> Resistor_SMD:R_0805_2012Metric
- R9: renamed from R4; footprint Resistor_THT:R_Axial_DIN0207_L6.3mm_D2.5mm_P7.62mm_Horizontal -> Resistor_SMD:R_0805_2012Metric
- Y1: footprint Crystal:Crystal_HC49-4H_Vertical -> Crystal:Crystal_SMD_HC49-SD
- renumbered J2 to J3, J3 to J4, J4 to J5, J5 to J6
Connections:
- net +5V: now also R5.1, R1.1, R2.1, R3.1, R4.1
- net BUZZ: now also U1.12 (PD6); no longer U1.11 (PD5)
- net DM1: now also U1.2 (PD0); no longer U1.23 (PC0)
- net DM2: now also U1.26 (PC3); no longer U1.14 (PB0)
- net GND: now also J2.10 (Pin_10), J2.6 (Pin_6), J2.7 (Pin_7), J2.8 (Pin_8), J2.9 (Pin_9); no longer R5.2
- net LED: now also U1.11 (PD5); no longer U1.15 (PB1)
- net PM2: now also U1.15 (PB1); no longer U1.12 (PD6)
- net RST1: no longer U1.1 (~{RESET}/PC6)
- net S1: now also U1.14 (PB0), J2.1 (Pin_1), R1.2; no longer R5.1, U1.13 (PD7)
- net S2: now also U1.13 (PD7), J2.2 (Pin_2), R2.2; no longer U1.24 (PC1)
- net S3: now also J2.3 (Pin_3), R3.2
- net S4: now also U1.24 (PC1), J2.4 (Pin_4), R4.2; no longer U1.26 (PC3)
- net S5: now also R5.2, U1.23 (PC0), J2.5 (Pin_5); no longer U1.2 (PD0)
- net RST2 renamed RST
- net RST: now also U1.1 (~{RESET}/PC6)
Other:
- moved on the sheet: BZ1, C1, C2, C3, D1, D2, H1, H2, H3, H4, J1, J3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

Commit message: updated track width
Parts:
- C1: footprint Capacitor_SMD:CP_Elec_6.3x4.5 -> Capacitor_SMD:CP_Elec_4x3.9
Changed lines of the file:
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@@
       (effects (font (size 1.27 1.27)))
     )
-    (property "Footprint" "Capacitor_SMD:CP_Elec_6.3x4.5" (at 93.98 41.91 0)
+    (property "Footprint" "Capacitor_SMD:CP_Elec_4x3.9" (at 93.98 41.91 0)
       (effects (font (size 1.27 1.27)) hide)
     )
